File: PCB/combobreaker_v2_oki_78sr_eagle/ComboBreaker.brd (EAGLE design)
At the start: 60.9 x 39.4 mm, 15 parts

Commit message: Updated v2 Eagle PCB
* Renamed Stepper pinout labels
* Added ground connections
* Manually set MIN_DELAY
Parts:
- turned C1 to 0 degrees
Connections:
- net 1A_BLK renamed 1B_BLK
- net 1B_GRN renamed 1A_GRN
Routing:
- net GND: track 0.00 -> 16.0 mm
- net VCC: track 51.4 -> 50.7 mm
Changed lines of the file:
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@@
 <text x="60.579" y="30.861" size="0.6096" layer="21" font="vector" rot="R90">2A</text>
 <text x="60.579" y="28.321" size="0.6096" layer="21" font="vector" rot="R90">2B</text>
-<text x="60.579" y="33.401" size="0.6096" layer="21" font="vector" rot="R90">1B</text>
-<text x="60.579" y="35.941" size="0.6096" layer="21" font="vector" rot="R90">1A</text>
+<text x="60.579" y="33.401" size="0.6096" layer="21" font="vector" rot="R90">1A</text>
+<text x="60.579" y="35.941" size="0.6096" layer="21" font="vector" rot="R90">1B</text>
 <wire x1="47.879" y1="30.734" x2="47.879" y2="29.972" width="0.127" layer="21"/>
 <wire x1="48.26" y1="30.353" x2="47.498" y2="30.353" width="0.127" layer="21"/>
@@
 <attribute name="VALUE" x="13.967715625" y="8.197671875" size="0.762" layer="21" font="vector"/>
 </element>
-<element name="C1" library="resistor" package="E3,5-8" value="100uF" x="45.72188125" y="24.3779" smashed="yes" rot="R180">
-<attribute name="VALUE" x="44.18828125" y="26.559109375" size="0.762" layer="21" ratio="10"/>
+<element name="C1" library="resistor" package="E3,5-8" value="100uF" x="45.7547625" y="24.37138125" smashed="yes">
+<attribute name="VALUE" x="47.669321875" y="22.395471875" size="0.762" layer="21" ratio="10" rot="R180"/>
 </element>
 <element name="OKI-78SR" library="carrilib" package="OKI-78SRH" value="5/1.5-W36H-C" x="34.671" y="25.527" smashed="yes" rot="R180">
@@
 <wire x1="13.97" y1="33.401" x2="13.97" y2="34.798" width="0.6096" layer="16"/>
 </signal>
-<signal name="1B_GRN">
+<signal name="1A_GRN">
 <contactref element="STEPPER" pad="3"/>
 <contactref element="A4988" pad="1A"/>
@@
 <contactref element="PWR" pad="1"/>
 <contactref element="DISPLAY" pad="1"/>
-<wire x1="43.94388125" y1="24.3779" x2="44.466" y2="31.733" width="0" layer="19" extent="1-1"/>
+<wire x1="44.466" y1="31.733" x2="44.45" y2="31.733" width="0.4064" layer="1"/>
+<wire x1="44.45" y1="31.733" x2="44.45" y2="34.29" width="0.4064" layer="1"/>
+<wire x1="44.45" y1="34.29" x2="44.9508125" y2="34.783578125" width="0.4064" layer="1"/>
+<wire x1="44.9508125" y1="34.783578125" x2="47.129621875" y2="34.755575" width="0.4064" layer="1"/>
+<wire x1="47.129621875" y1="34.755575" x2="47.53221875" y2="34.346" width="0.4064" layer="1"/>
+<wire x1="47.53221875" y1="25.15461875" x2="47.5327625" y2="24.37138125" width="0.4064" layer="1"/>
+<wire x1="47.53221875" y1="34.346" x2="47.53221875" y2="25.15461875" width="0.4064" layer="1"/>
 </signal>
 <signal name="2A_RED">
@@
 <wire x1="57.912" y1="31.369" x2="58.42" y2="31.369" width="0.6096" layer="16"/>
 </signal>
-<signal name="1A_BLK">
+<signal name="1B_BLK">
 <contactref element="STEPPER" pad="4"/>
 <contactref element="A4988" pad="1B"/>
@@
 <contactref element="A4988" pad="VMOT"/>
 <contactref element="PWR" pad="2"/>
-<wire x1="46.466" y1="27.956" x2="46.466" y2="31.733" width="0.8128" layer="1"/>
-<wire x1="47.49988125" y1="24.3779" x2="47.49988125" y2="26.79511875" width="0.8128" layer="1"/>
-<wire x1="46.482" y1="27.94" x2="47.49988125" y2="26.79511875" width="0.8128" layer="1"/>
-<wire x1="46.482" y1="27.94" x2="46.466" y2="27.956" width="0.8128" layer="1"/>
+<wire x1="46.466" y1="29.226" x2="46.466" y2="31.733" width="0.8128" layer="1"/>
+<wire x1="43.9767625" y1="24.37138125" x2="43.964478125" y2="25.39416875" width="0.8128" layer="1"/>
+<wire x1="43.964478125" y1="25.39416875" x2="43.959421875" y2="25.815090625" width="0.8128" layer="1"/>
+<wire x1="45.212" y1="27.94" x2="46.466" y2="29.226" width="0.8128" layer="1"/>
 <wire x1="8.89" y1="34.798" x2="8.89" y2="35.56" width="0.8128" layer="16"/>
 <wire x1="8.89" y1="35.56" x2="10.16" y2="36.83" width="0.8128" layer="16"/>
@@
 <wire x1="32.131" y1="35.687" x2="32.131" y2="33.909" width="0.8128" layer="1"/>
 <wire x1="32.131" y1="33.909" x2="38.1" y2="27.94" width="0.8128" layer="1"/>
-<wire x1="38.1" y1="27.94" x2="46.482" y2="27.94" width="0.8128" layer="1"/>
+<wire x1="43.6972875" y1="27.94" x2="38.1" y2="27.94" width="0.8128" layer="1"/>
+<wire x1="43.6972875" y1="27.94" x2="45.212" y2="27.94" width="0.8128" layer="1"/>
+<wire x1="43.964478125" y1="25.39416875" x2="43.964478125" y2="27.672809375" width="0.8128" layer="1"/>
+<wire x1="43.964478125" y1="27.672809375" x2="43.6972875" y2="27.94" width="0.4064" layer="1"/>
 </signal>
 <signal name="N$2">

Commit message: Updated ComboBreaker.ino code
* Corrected DIR and STEP pins
* Added delayMicroseconds(MIN_DELAY); to line 362 which resolved the
issue with the stepper motor not stepping correctly
Parts:
- removed PWR: 7-35v, SparkFun-Connectors:JST-2-SMD
- added J1: (no value), SparkFun-Connectors:JST-2-SMD
Connections:
- net GND: now also J1.1; no longer PWR.1
- net VCC: now also J1.2; no longer PWR.2
Changed lines of the file:
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@@
 <attribute name="VALUE" x="11.684" y="27.432" size="0.6096" layer="21"/>
-</element>
-<element name="PWR" library="SparkFun-Connectors" package="JST-2-SMD" value="7-35v" x="45.466" y="35.433" smashed="yes">
-<attribute name="NAME" x="44.45" y="36.195" size="0.8128" layer="25" font="vector" ratio="15"/>
-<attribute name="PROD_ID" value="CONN-11443" x="45.466" y="35.433" size="1.778" layer="27" display="off"/>
-<attribute name="SF_ID" value="PRT-08612" x="45.466" y="35.433" size="1.778" layer="27" display="off"/>
-<attribute name="VALUE" x="44.196" y="34.925" size="0.6096" layer="21" font="vector" ratio="10"/>
 </element>
 <element name="DISPLAY" library="SparkFun-Connectors" package="1X04" value="I2C" x="2.032" y="23.622" smashed="yes" rot="R270">
@@
 <element name="U$5" library="Aidan" package="AM" value="" x="52.832" y="27.813" rot="R90"/>
 <element name="U$6" library="Aidan" package="MASTERLOCK2" value="" x="48.133" y="33.02" rot="MR0"/>
+<element name="J1" library="SparkFun-Connectors" package="JST-2-SMD" value="" x="45.4715125" y="35.439634375">
+<attribute name="PROD_ID" value="CONN-11443" x="45.4715125" y="35.439634375" size="1.778" layer="27" display="off"/>
+<attribute name="SF_ID" value="PRT-08612" x="45.4715125" y="35.439634375" size="1.778" layer="27" display="off"/>
+</element>
 </elements>
 <signals>
@@
 <contactref element="A4988" pad="GND@0"/>
 <contactref element="A4988" pad="GND"/>
-<contactref element="PWR" pad="1"/>
 <contactref element="DISPLAY" pad="1"/>
-<wire x1="44.466" y1="31.733" x2="44.45" y2="31.733" width="0.4064" layer="1"/>
 <wire x1="44.45" y1="31.733" x2="44.45" y2="34.29" width="0.4064" layer="1"/>
 <wire x1="44.45" y1="34.29" x2="44.9508125" y2="34.783578125" width="0.4064" layer="1"/>
-<wire x1="44.9508125" y1="34.783578125" x2="47.129621875" y2="34.755575" width="0.4064" layer="1"/>
-<wire x1="47.129621875" y1="34.755575" x2="47.53221875" y2="34.346" width="0.4064" layer="1"/>
+<wire x1="44.9508125" y1="34.783578125" x2="47.07330625" y2="34.781178125" width="0.4064" layer="1"/>
+<wire x1="47.07330625" y1="34.781178125" x2="47.53221875" y2="34.346" width="0.4064" layer="1"/>
 <wire x1="47.53221875" y1="25.15461875" x2="47.5327625" y2="24.37138125" width="0.4064" layer="1"/>
 <wire x1="47.53221875" y1="34.346" x2="47.53221875" y2="25.15461875" width="0.4064" layer="1"/>
+<contactref element="J1" pad="1"/>
+<wire x1="44.45" y1="31.733" x2="44.4715125" y2="31.739634375" width="0" layer="19" extent="1-1"/>
 </signal>
 <signal name="2A_RED">
@@
 <contactref element="OKI-78SR" pad="1"/>
 <contactref element="A4988" pad="VMOT"/>
-<contactref element="PWR" pad="2"/>
-<wire x1="46.466" y1="29.226" x2="46.466" y2="31.733" width="0.8128" layer="1"/>
 <wire x1="43.9767625" y1="24.37138125" x2="43.964478125" y2="25.39416875" width="0.8128" layer="1"/>
 <wire x1="43.964478125" y1="25.39416875" x2="43.959421875" y2="25.815090625" width="0.8128" layer="1"/>
@@
 <wire x1="43.964478125" y1="25.39416875" x2="43.964478125" y2="27.672809375" width="0.8128" layer="1"/>
 <wire x1="43.964478125" y1="27.672809375" x2="43.6972875" y2="27.94" width="0.4064" layer="1"/>
+<contactref element="J1" pad="2"/>
+<wire x1="46.466" y1="29.226" x2="46.466" y2="31.734121875" width="0.8128" layer="1"/>
+<wire x1="46.466" y1="31.734121875" x2="46.4715125" y2="31.739634375" width="0.4064" layer="1"/>
 </signal>
 <signal name="N$2">

Commit message: Added GND pour to TOP layer
*** Added GND pour to TOP layer to resolve issues with SMD JST connector etc.
*** Adjusted JST connector pin name to GND.
Routing:
- net GND: track 16.0 -> 0.00 mm
- added copper zone on layer 1, net GND
Changed lines of the file:
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@@
 <?xml version="1.0" encoding="utf-8"?>
 <!DOCTYPE eagle SYSTEM "eagle.dtd">
-<eagle version="8.1.0">
+<eagle version="8.3.2">
 <drawing>
 <settings>
 <setting alwaysvectorfont="yes"/>
+<setting keepoldvectorfont="yes"/>
 <setting verticaltext="up"/>
 </settings>
@@
 </autorouter>
 <elements>
-<element name="SERVO" library="con-lstb" package="MA04-1" value="S1213" x="58.42" y="6.35" smashed="yes" rot="R90">
+<element name="SERVO" library="con-lstb" library_urn="urn:adsk.eagle:library:162" package="MA04-1" package3d_urn="urn:adsk.eagle:package:8337/1" value="S1213" x="58.42" y="6.35" smashed="yes" rot="R90">
 <attribute name="MF" value="" x="58.42" y="6.35" size="1.778" layer="27" rot="R90" display="off"/>
 <attribute name="MPN" value="" x="58.42" y="6.35" size="1.778" layer="27" rot="R90" display="off"/>
@@
 <attribute name="VALUE" x="56.769" y="5.08" size="0.6096" layer="21" rot="R90"/>
 </element>
-<element name="STEPPER" library="con-lstb" package="MA04-1" value="28STH32" x="58.42" y="32.639" smashed="yes" rot="R90">
+<element name="STEPPER" library="con-lstb" library_urn="urn:adsk.eagle:library:162" package="MA04-1" package3d_urn="urn:adsk.eagle:package:8337/1" value="28STH32" x="58.42" y="32.639" smashed="yes" rot="R90">
 <attribute name="MF" value="" x="58.42" y="32.639" size="1.778" layer="27" rot="R90" display="off"/>
 <attribute name="MPN" value="" x="58.42" y="32.639" size="1.778" layer="27" rot="R90" display="off"/>
@@
 <attribute name="VALUE" x="56.642" y="32.766" size="0.6096" layer="21" ratio="10" rot="R90"/>
 </element>
-<element name="ENCODER" library="con-lstb" package="MA05-1" value="HKT22" x="58.42" y="19.431" smashed="yes" rot="R90">
+<element name="ENCODER" library="con-lstb" library_urn="urn:adsk.eagle:library:162" package="MA05-1" package3d_urn="urn:adsk.eagle:package:8332/1" value="HKT22" x="58.42" y="19.431" smashed="yes" rot="R90">
 <attribute name="MF" value="" x="58.42" y="19.431" size="1.778" layer="27" rot="R90" display="off"/>
 <attribute name="MPN" value="" x="58.42" y="19.431" size="1.778" layer="27" rot="R90" display="off"/>
@@
 <attribute name="VALUE" x="13.967715625" y="8.197671875" size="0.762" layer="21" font="vector"/>
 </element>
-<element name="C1" library="resistor" package="E3,5-8" value="100uF" x="45.7547625" y="24.37138125" smashed="yes">
+<element name="C1" library="resistor" library_urn="urn:adsk.eagle:library:348" package="E3,5-8" package3d_urn="urn:adsk.eagle:package:25842/1" value="100uF" x="45.7547625" y="24.37138125" smashed="yes">
 <attribute name="VALUE" x="47.669321875" y="22.395471875" size="0.762" layer="21" ratio="10" rot="R180"/>
 </element>
@@
 <contactref element="A4988" pad="GND"/>
 <contactref element="DISPLAY" pad="1"/>
-<wire x1="44.45" y1="31.733" x2="44.45" y2="34.29" width="0.4064" layer="1"/>
-<wire x1="44.45" y1="34.29" x2="44.9508125" y2="34.783578125" width="0.4064" layer="1"/>
-<wire x1="44.9508125" y1="34.783578125" x2="47.07330625" y2="34.781178125" width="0.4064" layer="1"/>
-<wire x1="47.07330625" y1="34.781178125" x2="47.53221875" y2="34.346" width="0.4064" layer="1"/>
-<wire x1="47.53221875" y1="25.15461875" x2="47.5327625" y2="24.37138125" width="0.4064" layer="1"/>
-<wire x1="47.53221875" y1="34.346" x2="47.53221875" y2="25.15461875" width="0.4064" layer="1"/>
 <contactref element="J1" pad="1"/>
-<wire x1="44.45" y1="31.733" x2="44.4715125" y2="31.739634375" width="0" layer="19" extent="1-1"/>
+<polygon width="0.127" layer="1">
+<vertex x="0" y="39.37"/>
+<vertex x="60.96" y="39.37"/>
+<vertex x="60.96" y="0"/>
+<vertex x="0" y="0"/>
+</polygon>
 </signal>
 <signal name="2A_RED">
@@
 which will not be processed correctly with this version.
 </note>
+<note version="8.2" severity="warning">
+Since Version 8.2, EAGLE supports online libraries. The ids
+of those online libraries will not be understood (or retained)
+with this version.
+</note>
+<note version="8.3" severity="warning">
+Since Version 8.3, EAGLE supports URNs for individual library
+assets (packages, symbols, and devices). The URNs of those assets
+will not be understood (or retained) with this version.
+</note>
+<note version="8.3" severity="warning">
+Since Version 8.3, EAGLE supports the association of 3D packages
+with devices in libraries, schematics, and board files. Those 3D
+packages will not be understood (or retained) with this version.
+</note>
 </compatibility>

Commit message: Minor changes to schematic
Parts:
- PWR: value (none) -> 7-35v
- turned C1 to 180 degrees
- renumbered J1 to PWR
Routing:
- net VCC: track 50.7 -> 51.4 mm
Changed lines of the file:
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@@
 <attribute name="VALUE" x="13.967715625" y="8.197671875" size="0.762" layer="21" font="vector"/>
 </element>
-<element name="C1" library="resistor" library_urn="urn:adsk.eagle:library:348" package="E3,5-8" package3d_urn="urn:adsk.eagle:package:25842/1" value="100uF" x="45.7547625" y="24.37138125" smashed="yes">
-<attribute name="VALUE" x="47.669321875" y="22.395471875" size="0.762" layer="21" ratio="10" rot="R180"/>
+<element name="C1" library="resistor" library_urn="urn:adsk.eagle:library:348" package="E3,5-8" package3d_urn="urn:adsk.eagle:package:25842/1" value="100uF" x="45.7547625" y="24.37138125" smashed="yes" rot="R180">
+<attribute name="VALUE" x="44.319434375" y="21.58788125" size="0.762" layer="21" ratio="10"/>
 </element>
 <element name="OKI-78SR" library="carrilib" package="OKI-78SRH" value="5/1.5-W36H-C" x="34.671" y="25.527" smashed="yes" rot="R180">
@@
 <element name="U$5" library="Aidan" package="AM" value="" x="52.832" y="27.813" rot="R90"/>
 <element name="U$6" library="Aidan" package="MASTERLOCK2" value="" x="48.133" y="33.02" rot="MR0"/>
-<element name="J1" library="SparkFun-Connectors" package="JST-2-SMD" value="" x="45.4715125" y="35.439634375">
+<element name="PWR" library="SparkFun-Connectors" package="JST-2-SMD" value="7-35v" x="45.4715125" y="35.439634375" smashed="yes">
+<attribute name="NAME" x="44.17718125" y="36.361628125" size="1.016" layer="25" font="vector" ratio="20"/>
 <attribute name="PROD_ID" value="CONN-11443" x="45.4715125" y="35.439634375" size="1.778" layer="27" display="off"/>
 <attribute name="SF_ID" value="PRT-08612" x="45.4715125" y="35.439634375" size="1.778" layer="27" display="off"/>
+<attribute name="VALUE" x="44.19696875" y="35.115903125" size="0.6096" layer="27" font="vector" ratio="20"/>
 </element>
 </elements>
@@
 <contactref element="A4988" pad="GND"/>
 <contactref element="DISPLAY" pad="1"/>
-<contactref element="J1" pad="1"/>
 <polygon width="0.127" layer="1">
 <vertex x="0" y="39.37"/>
@@
 <vertex x="0" y="0"/>
 </polygon>
+<contactref element="PWR" pad="1"/>
 </signal>
 <signal name="2A_RED">
@@
 <contactref element="OKI-78SR" pad="1"/>
 <contactref element="A4988" pad="VMOT"/>
-<wire x1="43.9767625" y1="24.37138125" x2="43.964478125" y2="25.39416875" width="0.8128" layer="1"/>
-<wire x1="43.964478125" y1="25.39416875" x2="43.959421875" y2="25.815090625" width="0.8128" layer="1"/>
-<wire x1="45.212" y1="27.94" x2="46.466" y2="29.226" width="0.8128" layer="1"/>
+<wire x1="45.212" y1="27.94" x2="46.4678125" y2="27.937253125" width="0.8128" layer="1"/>
+<wire x1="46.4678125" y1="27.937253125" x2="46.465590625" y2="29.224778125" width="0.8128" layer="1"/>
+<wire x1="46.465590625" y1="29.224778125" x2="46.466" y2="30.496" width="0.8128" layer="1"/>
 <wire x1="8.89" y1="34.798" x2="8.89" y2="35.56" width="0.8128" layer="16"/>
 <wire x1="8.89" y1="35.56" x2="10.16" y2="36.83" width="0.8128" layer="16"/>
@@
 <wire x1="32.131" y1="35.687" x2="32.131" y2="33.909" width="0.8128" layer="1"/>
 <wire x1="32.131" y1="33.909" x2="38.1" y2="27.94" width="0.8128" layer="1"/>
-<wire x1="43.6972875" y1="27.94" x2="38.1" y2="27.94" width="0.8128" layer="1"/>
-<wire x1="43.6972875" y1="27.94" x2="45.212" y2="27.94" width="0.8128" layer="1"/>
-<wire x1="43.964478125" y1="25.39416875" x2="43.964478125" y2="27.672809375" width="0.8128" layer="1"/>
-<wire x1="43.964478125" y1="27.672809375" x2="43.6972875" y2="27.94" width="0.4064" layer="1"/>
-<contactref element="J1" pad="2"/>
-<wire x1="46.466" y1="29.226" x2="46.466" y2="31.734121875" width="0.8128" layer="1"/>
+<wire x1="45.212" y1="27.94" x2="38.1" y2="27.94" width="0.8128" layer="1"/>
+<contactref element="PWR" pad="2"/>
+<wire x1="46.466" y1="30.496" x2="46.466" y2="31.734121875" width="0.8128" layer="1"/>
 <wire x1="46.466" y1="31.734121875" x2="46.4715125" y2="31.739634375" width="0.4064" layer="1"/>
+<wire x1="47.539503125" y1="26.776896875" x2="47.5327625" y2="24.37138125" width="0.8128" layer="1"/>
+<wire x1="46.4678125" y1="27.937253125" x2="47.539503125" y2="26.776896875" width="0.8128" layer="1"/>
 </signal>
 <signal name="N$2">

Commit message: Updated header pins to circles from ovals
Parts:
- ENCODER: device con-lstb:MA05-1 -> ComboBreaker:CON-LSTB_MA05-1
- SERVO, STEPPER: device con-lstb:MA04-1 -> ComboBreaker:ADAFRUIT_1X04-BIG
- moved STEPPER 3.81 mm to (58.4, 28.8)
- moved SERVO 3.81 mm to (58.4, 2.54)
Changed lines of the file:
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@@
 </autorouter>
 <elements>
-<element name="SERVO" library="con-lstb" library_urn="urn:adsk.eagle:library:162" package="MA04-1" package3d_urn="urn:adsk.eagle:package:8337/1" value="S1213" x="58.42" y="6.35" smashed="yes" rot="R90">
-<attribute name="MF" value="" x="58.42" y="6.35" size="1.778" layer="27" rot="R90" display="off"/>
-<attribute name="MPN" value="" x="58.42" y="6.35" size="1.778" layer="27" rot="R90" display="off"/>
+<element name="SERVO" library="ComboBreaker" package="ADAFRUIT_1X04-BIG" value="S1213" x="58.42" y="2.54" smashed="yes" rot="R90">
 <attribute name="NAME" x="56.8452" y="1.1938" size="0.762" layer="25" ratio="15" rot="R90"/>
-<attribute name="OC_FARNELL" value="unknown" x="58.42" y="6.35" size="1.778" layer="27" rot="R90" display="off"/>
-<attribute name="OC_NEWARK" value="unknown" x="58.42" y="6.35" size="1.778" layer="27" rot="R90" display="off"/>
 <attribute name="VALUE" x="56.769" y="5.08" size="0.6096" layer="21" rot="R90"/>
 </element>
-<element name="STEPPER" library="con-lstb" library_urn="urn:adsk.eagle:library:162" package="MA04-1" package3d_urn="urn:adsk.eagle:package:8337/1" value="28STH32" x="58.42" y="32.639" smashed="yes" rot="R90">
-<attribute name="MF" value="" x="58.42" y="32.639" size="1.778" layer="27" rot="R90" display="off"/>
-<attribute name="MPN" value="" x="58.42" y="32.639" size="1.778" layer="27" rot="R90" display="off"/>
+<element name="STEPPER" library="ComboBreaker" package="ADAFRUIT_1X04-BIG" value="28STH32" x="58.42" y="28.829" smashed="yes" rot="R90">
 <attribute name="NAME" x="56.7182" y="27.4828" size="0.762" layer="25" ratio="15" rot="R90"/>
-<attribute name="OC_FARNELL" value="unknown" x="58.42" y="32.639" size="1.778" layer="27" rot="R90" display="off"/>
-<attribute name="OC_NEWARK" value="unknown" x="58.42" y="32.639" size="1.778" layer="27" rot="R90" display="off"/>
 <attribute name="VALUE" x="56.642" y="32.766" size="0.6096" layer="21" ratio="10" rot="R90"/>
 </element>
-<element name="ENCODER" library="con-lstb" library_urn="urn:adsk.eagle:library:162" package="MA05-1" package3d_urn="urn:adsk.eagle:package:8332/1" value="HKT22" x="58.42" y="19.431" smashed="yes" rot="R90">
+<element name="ENCODER" library="ComboBreaker" package="CON-LSTB_MA05-1" value="HKT22" x="58.42" y="19.431" smashed="yes" rot="R90">
 <attribute name="MF" value="" x="58.42" y="19.431" size="1.778" layer="27" rot="R90" display="off"/>
 <attribute name="MPN" value="" x="58.42" y="19.431" size="1.778" layer="27" rot="R90" display="off"/>
