File: PCB/combobreaker_v2_oki_78sr_eagle/ComboBreaker.brd (EAGLE design)
At the start: 60.9 x 39.4 mm, 15 parts

Commit message: Updated drill size to .35
* Updated drill sizes on most holes to .35
* Adjusted Mini-B USB connector outline on Arduino Nano silkscreen
Connections:
- net GND: now also PWR.GND; no longer PWR.1
Changed lines of the file:
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@@
 <wire x1="55.88" y1="32.639" x2="55.88" y2="36.703" width="0.0762" layer="21"/>
 <wire x1="55.88" y1="5.08" x2="55.88" y2="7.874" width="0.0762" layer="21"/>
-<wire x1="4.572" y1="14.097" x2="4.572" y2="25.527" width="0.0762" layer="21"/>
+<wire x1="4.572" y1="15.033059375" x2="4.572" y2="24.45721875" width="0.0762" layer="21"/>
 <text x="25.146" y="26.543" size="0.8128" layer="22" font="vector" rot="MR0">PCB:</text>
 <text x="22.098" y="26.543" size="1.27" layer="22" font="vector" ratio="20" rot="MR0">Aidan McCarthy</text>
@@
 </element>
 <element name="ARDUINO" library="ArduinoNanoV30" package="ARDUINO_NANO" value="Arduino Nano V3.0 Module" x="25.397715625" y="10.102671875" smashed="yes">
-<attribute name="NAME" x="13.967715625" y="9.467671875" size="1.27" layer="21" font="vector" ratio="10"/>
-<attribute name="VALUE" x="13.967715625" y="8.197671875" size="0.762" layer="21" font="vector"/>
+<attribute name="NAME" x="16.09986875" y="10.4952625" size="1.27" layer="21" font="vector" ratio="10"/>
+<attribute name="VALUE" x="16.139353125" y="8.632421875" size="0.762" layer="21" font="vector"/>
 </element>
 <element name="C1" library="resistor" library_urn="urn:adsk.eagle:library:348" package="E3,5-8" package3d_urn="urn:adsk.eagle:package:25842/1" value="100uF" x="45.7547625" y="24.37138125" smashed="yes" rot="R180">
@@
 </element>
 <element name="DISPLAY" library="SparkFun-Connectors" package="1X04" value="I2C" x="2.032" y="23.622" smashed="yes" rot="R270">
-<attribute name="NAME" x="5.715" y="14.097" size="0.8128" layer="25" font="vector" ratio="15" rot="R90"/>
-<attribute name="VALUE" x="4.826" y="25.527" size="0.8128" layer="21" font="vector" ratio="15" rot="R270"/>
+<attribute name="NAME" x="5.715" y="15.367" size="0.8128" layer="25" font="vector" ratio="15" rot="R90"/>
+<attribute name="VALUE" x="4.826" y="24.257" size="0.8128" layer="21" font="vector" ratio="15" rot="R270"/>
 </element>
 <element name="U$1" library="SparkFun-Hardware" package="STAND-OFF" value="" x="3.304796875" y="3.19950625" smashed="yes">
@@
 <polygon width="0.4064" layer="16">
 <vertex x="60.96180625" y="1.3426625"/>
-<vertex x="60.926571875" y="39.41236875"/>
-<vertex x="0.045315625" y="39.4118875"/>
-<vertex x="0.074646875" y="1.291865625" curve="90.08677"/>
-<vertex x="1.504003125" y="-0.00775"/>
+<vertex x="60.9277875" y="38.098921875" curve="89.947341"/>
+<vertex x="59.61191875" y="39.412359375"/>
+<vertex x="1.632096875" y="39.4119" curve="90.240865"/>
+<vertex x="0.0465375" y="37.823890625"/>
+<vertex x="0.074615625" y="1.332365625" curve="89.961499"/>
+<vertex x="1.414325" y="-0.007759375"/>
 <vertex x="59.61815" y="-0.002034375" curve="89.906409"/>
 </polygon>
@@
 <contactref element="DISPLAY" pad="1"/>
 <polygon width="0.127" layer="1">
-<vertex x="0" y="39.37"/>
-<vertex x="60.96" y="39.37"/>
-<vertex x="60.96" y="0"/>
-<vertex x="0" y="0"/>
+<vertex x="0" y="1.27"/>
+<vertex x="0" y="38.1" curve="-90"/>
+<vertex x="1.27" y="39.37"/>
+<vertex x="59.69" y="39.37" curve="-90"/>
+<vertex x="60.96" y="38.1"/>
+<vertex x="60.96" y="1.27" curve="-90"/>
+<vertex x="59.69" y="0"/>
+<vertex x="1.27" y="0" curve="-90"/>
 </polygon>
-<contactref element="PWR" pad="1"/>
+<contactref element="PWR" pad="GND"/>
 </signal>
 <signal name="2A_RED">
@@
 <signal name="N$4">
 <polygon width="0.4064" layer="1">
-<vertex x="0" y="13.97"/>
+<vertex x="0" y="38.1"/>
 <vertex x="0" y="1.27" curve="90"/>
 <vertex x="1.27" y="0"/>
@@
 <vertex x="59.69" y="39.37"/>
 <vertex x="1.27" y="39.37" curve="90"/>
-<vertex x="0" y="38.1"/>
 </polygon>
 </signal>

Commit message: v3 PCB
Minor changes
V3 send to fabrication
Parts:
- removed C1: 100uF, resistor:E3,5-8
- added C2: 100uF, resistor:E3,5-8
Connections:
- net GND: now also C2.-; no longer C1.-
- net VCC: now also C2.+; no longer C1.+
Changed lines of the file:
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@@
 </element>
 <element name="ARDUINO" library="ArduinoNanoV30" package="ARDUINO_NANO" value="Arduino Nano V3.0 Module" x="25.397715625" y="10.102671875" smashed="yes">
-<attribute name="NAME" x="16.09986875" y="10.4952625" size="1.27" layer="21" font="vector" ratio="10"/>
-<attribute name="VALUE" x="16.139353125" y="8.632421875" size="0.762" layer="21" font="vector"/>
-</element>
-<element name="C1" library="resistor" library_urn="urn:adsk.eagle:library:348" package="E3,5-8" package3d_urn="urn:adsk.eagle:package:25842/1" value="100uF" x="45.7547625" y="24.37138125" smashed="yes" rot="R180">
-<attribute name="VALUE" x="44.319434375" y="21.58788125" size="0.762" layer="21" ratio="10"/>
+<attribute name="NAME" x="20.309028125" y="10.475121875" size="1.27" layer="21" font="vector" ratio="10"/>
+<attribute name="VALUE" x="16.17963125" y="9.45819375" size="0.762" layer="21" font="vector"/>
 </element>
 <element name="OKI-78SR" library="carrilib" package="OKI-78SRH" value="5/1.5-W36H-C" x="34.671" y="25.527" smashed="yes" rot="R180">
@@
 <attribute name="SF_ID" value="PRT-08612" x="45.4715125" y="35.439634375" size="1.778" layer="27" display="off"/>
 <attribute name="VALUE" x="44.19696875" y="35.115903125" size="0.6096" layer="27" font="vector" ratio="20"/>
+</element>
+<element name="C2" library="resistor" library_urn="urn:adsk.eagle:library:348" package="E3,5-8" package3d_urn="urn:adsk.eagle:package:25842/1" value="100uF" x="45.77054375" y="24.427296875" smashed="yes" rot="R180">
+<attribute name="VALUE" x="47.71498125" y="27.287403125" size="0.8128" layer="27" font="vector" ratio="10" rot="R180"/>
 </element>
 </elements>
@@
 <contactref element="ARDUINO" pad="19"/>
 <contactref element="ARDUINO" pad="14"/>
-<contactref element="C1" pad="-"/>
 <contactref element="SERVO" pad="1"/>
 <contactref element="OKI-78SR" pad="2"/>
@@
 </polygon>
 <contactref element="PWR" pad="GND"/>
+<contactref element="C2" pad="-"/>
 </signal>
 <signal name="2A_RED">
@@
 </signal>
 <signal name="VCC">
-<contactref element="C1" pad="+"/>
 <contactref element="OKI-78SR" pad="1"/>
 <contactref element="A4988" pad="VMOT"/>
@@
 <wire x1="46.466" y1="30.496" x2="46.466" y2="31.734121875" width="0.8128" layer="1"/>
 <wire x1="46.466" y1="31.734121875" x2="46.4715125" y2="31.739634375" width="0.4064" layer="1"/>
-<wire x1="47.539503125" y1="26.776896875" x2="47.5327625" y2="24.37138125" width="0.8128" layer="1"/>
 <wire x1="46.4678125" y1="27.937253125" x2="47.539503125" y2="26.776896875" width="0.8128" layer="1"/>
+<contactref element="C2" pad="+"/>
+<wire x1="47.539503125" y1="26.776896875" x2="47.54854375" y2="24.427296875" width="0.8128" layer="1"/>
 </signal>
 <signal name="N$2">
